File: inverter-1kw.sch (EAGLE design)
At the start: 240 parts, among them IC1 LM358D, IC5 ISO3082, IC6 25LC080SN, IC9 LM358D, Q2 1200980569**TRANS SMD NPN MMB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, Q3 1200980569**TRANS SMD NPN MMB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, Q4 1200980569**TRANS SMD NPN MMB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, Q6 1200980569**TRANS SMD NPN MMB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, U1 ACS712, U2 STM32F334C6, U3 1039-2088**AM1L-0505SH30-NZ A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, U4 ACS712, U5 SI8230, U6 SI8230, U7 ACS712, X1 MCV3, X2 RADE2, X3 RADE2, X7 RADE2, X8 RADE2

Commit message: Giriş kondansatörleri düzenlendi.
Connections:
- removed net 400V-: U4.IP1-, U4.IP2-, X8.1, X8.2
- new net N$31: R94.1, R95.2
- new net N$32: R95.1, R96.2
- new net N$4: R93.1, R94.2
- new net V+: C83.1, C84.1, GN1.D, R65.2, R72.2, R74.2, R93.2, U4.IP1-, U4.IP2-
- net AGND: now also R96.1, X8.1, X8.2; no longer U4.IP1+, U4.IP2+
- net V_IN: now also U4.IP1+, U4.IP2+; no longer C83.1, C84.1, GN1.D, R65.2, R72.2, R74.2
Other:
- moved on the sheet: C31, C32, C33, C34, C35, C40, C72, C73, D1, D2, Q4, Q6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

Commit message: Bobin paketleri guncellendi. Roleler ince secildi.
Parts:
- added R97, R98: (no value), rcl:R-EU_R1206
- L1, L2: value SFT830D -> SFT1240; device inductors:SFT830D -> inductors:SFT1240
- RL1, RL2: value G5LE-TEK -> 0417; device Erelay:G5LE-TEK -> Erelay:0417
Connections:
- net N$32 renamed VIN_SENS
- removed net I_LEFT_AC: R47.1, U1.VO, U7.VO
- new net IA_SENS: U7.VO
- new net IB_SENS: R47.1, U1.VO
- new net VA_SENS: R25.1, R98.1
- new net VB_SENS: R87.1, R97.2
- net +12V: now also RL1G$1.1, RL2G$1.1; no longer RL1G$2.1, RL2G$2.1
- net AGND: now also R97.1, R98.2
- net N$28: now also R87.2; no longer R87.1
- net N$44: now also RL1G$1.2; no longer RL1G$2.2
- net N$51: now also RL2G$1.2; no longer RL2G$2.2
- net N$55: now also RL1G$2.P; no longer RL1G$1.S
- net VDIG+: now also RL1G$2.S, RL2G$2.S; no longer RL1G$1.P, RL2G$1.S
- net V_IN: now also RL2G$2.P; no longer RL2G$1.P
Other:
- note removed: "asdads"
- moved on the sheet: D1, D2, Q4, Q6, R24, R25, R36, R41, R57, R87, R94, R95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

Commit message: Role beslemeleri VDD ile sembolize edildi.
Connections:
- net +12V renamed VDD
- net VDIG+ renamed VSUPPLY+
- removed net V+: C83.1, C84.1, GN1.D, R65.2, R72.2, R74.2, R93.2, U4.IP1-, U4.IP2-
- new net IIN_SENS: U4.VO
- new net VIN: C83.1, C84.1, C95.1, C96.1, GN1.D, GN3.D, R65.2, R72.2, R74.2, R89.2, R91.2, R92.2, R93.2, U4.IP1-, U4.IP2-
- net I_LEFT_DC: no longer U4.VO
- net V_IN: no longer C95.1, C96.1, GN3.D, R89.2, R91.2, R92.2
Other:
- moved on the sheet: C114, C14, C15, C20, C21, C22, C23, C24, C38, C39, C43, C44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

Commit message: Cikis terminaline kondasator eklendi. Guc soketleri icin(4-pinli) kullanilacak urun linki value alanlarina yazildi.
Parts:
- added C11: (no value), capacitor-wima:C27/17
- X2, X3, X7, X8: value RADE2 -> https://ozdisan.com/connectors-and-interconnects/terminals/screw-connectors/K93-01AH
Connections:
- net N$1: now also C11.2
- net N$2: now also C11.1
Changed lines of the file:
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@@
 <layer number="250" name="Descript" color="3" fill="1" visible="no" active="no"/>
 <layer number="251" name="SMDround" color="12" fill="11" visible="no" active="no"/>
+<layer number="253" name="Extra" color="7" fill="1" visible="yes" active="yes"/>
 <layer number="254" name="cooling" color="7" fill="1" visible="yes" active="yes"/>
 <layer number="255" name="routoute" color="7" fill="1" visible="yes" active="yes"/>
@@
 <part name="GN3" library="my_parts1" deviceset="TP65H300G4LSG" device=""/>
 <part name="GN4" library="my_parts1" deviceset="TP65H300G4LSG" device=""/>
-<part name="L6" library="enko" deviceset="ARYA_COMMON_FILTER" device=""/>
-<part name="L7" library="enko" deviceset="ARYA_COMMON_FILTER" device=""/>
+<part name="L6" library="enko" library_urn="urn:adsk.eagle:library:26770947" deviceset="ARYA_COMMON_FILTER" device="" package3d_urn="urn:adsk.eagle:package:26773388/1"/>
+<part name="L7" library="enko" library_urn="urn:adsk.eagle:library:26770947" deviceset="ARYA_COMMON_FILTER" device="" package3d_urn="urn:adsk.eagle:package:26773388/1"/>
 <part name="DC1" library="my_parts1" deviceset="RI-0512S/P_DC_DC_5V_12V" device=""/>
 <part name="DC2" library="my_parts1" deviceset="RI-0512S/P_DC_DC_5V_12V" device=""/>
@@
 <part name="C35" library="rcl" deviceset="CPOL-EU" device="E7.5-18"/>
 <part name="C40" library="rcl" deviceset="CPOL-EU" device="E7.5-18"/>
-<part name="X7" library="enko" deviceset="RADE2" device=""/>
-<part name="X8" library="enko" deviceset="RADE2" device=""/>
+<part name="X7" library="enko" library_urn="urn:adsk.eagle:library:26770947" deviceset="RADE2" device="" package3d_urn="urn:adsk.eagle:package:26773267/1" value="https://ozdisan.com/connectors-and-interconnects/terminals/screw-connectors/K93-01AH"/>
+<part name="X8" library="enko" library_urn="urn:adsk.eagle:library:26770947" deviceset="RADE2" device="" package3d_urn="urn:adsk.eagle:package:26773267/1" value="https://ozdisan.com/connectors-and-interconnects/terminals/screw-connectors/K93-01AH"/>
 <part name="AGND3" library="supply1" library_urn="urn:adsk.eagle:library:371" deviceset="AGND" device=""/>
 <part name="AGND4" library="supply1" library_urn="urn:adsk.eagle:library:371" deviceset="AGND" device=""/>
@@
 <part name="C57" library="rcl" deviceset="C-EU" device="C1206" value="4.7u"/>
 <part name="+3V10" library="supply1" deviceset="+3V3" device=""/>
-<part name="IC5" library="enko" deviceset="ISO3082" device=""/>
+<part name="IC5" library="enko" library_urn="urn:adsk.eagle:library:26770947" deviceset="ISO3082" device="" package3d_urn="urn:adsk.eagle:package:26772954/1"/>
 <part name="C58" library="rcl" deviceset="C-EU" device="C0805" value="1200920113**CAP 0805 CER 100NF 50V %20 X7"/>
 <part name="SGND1" library="supply" deviceset="SGND" device=""/>
@@
 <part name="C74" library="rcl" deviceset="C-EU" device="C0805"/>
 <part name="SUPPLY62" library="supply2" deviceset="DGND" device=""/>
-<part name="L4" library="enko" deviceset="ACM2012-900--2P-T002" device=""/>
+<part name="L4" library="enko" library_urn="urn:adsk.eagle:library:26770947" deviceset="ACM2012-900--2P-T002" device="" package3d_urn="urn:adsk.eagle:package:26773148/1"/>
 <part name="D3" library="diode" deviceset="DIODE-" device="SOD323-W" value="https://www.digikey.com/product-detail/en/littelfuse-inc/AQ15C-01FTG/F10389CT-ND/7902217"/>
 <part name="D4" library="diode" deviceset="DIODE-" device="SOD323-W" value="https://www.digikey.com/product-detail/en/littelfuse-inc/AQ15C-01FTG/F10389CT-ND/7902217"/>
@@
 <part name="+3V4" library="supply1" deviceset="+3V3" device=""/>
 <part name="SUPPLY15" library="supply2" deviceset="+5V" device=""/>
-<part name="X2" library="enko" deviceset="RADE2" device=""/>
-<part name="X3" library="enko" deviceset="RADE2" device=""/>
+<part name="X2" library="enko" library_urn="urn:adsk.eagle:library:26770947" deviceset="RADE2" device="" package3d_urn="urn:adsk.eagle:package:26773267/1" value="https://ozdisan.com/connectors-and-interconnects/terminals/screw-connectors/K93-01AH"/>
+<part name="X3" library="enko" library_urn="urn:adsk.eagle:library:26770947" deviceset="RADE2" device="" package3d_urn="urn:adsk.eagle:package:26773267/1" value="https://ozdisan.com/connectors-and-interconnects/terminals/screw-connectors/K93-01AH"/>
 <part name="R23" library="rcl" library_urn="urn:adsk.eagle:library:334" deviceset="R-EU_" device="R1206" package3d_urn="urn:adsk.eagle:package:23540/2"/>
 <part name="R24" library="rcl" library_urn="urn:adsk.eagle:library:334" deviceset="R-EU_" device="R1206" package3d_urn="urn:adsk.eagle:package:23540/2"/>
@@
 <part name="VDD2" library="supply1" library_urn="urn:adsk.eagle:library:371" deviceset="VDD" device=""/>
 <part name="VDD3" library="supply1" library_urn="urn:adsk.eagle:library:371" deviceset="VDD" device=""/>
+<part name="C11" library="capacitor-wima" library_urn="urn:adsk.eagle:library:116" deviceset="C" device="27/17" package3d_urn="urn:adsk.eagle:package:5418/1"/>
 </parts>
 <sheets>
@@
 <attribute name="VALUE" x="71.12" y="386.08" size="1.778" layer="96" rot="R90"/>
 </instance>
+<instance part="C11" gate="G$1" x="786.13" y="172.72" smashed="yes">
+<attribute name="NAME" x="787.654" y="173.101" size="1.778" layer="95"/>
+<attribute name="VALUE" x="787.654" y="168.021" size="1.778" layer="96"/>
+</instance>
 </instances>
 <busses>
@@
 <junction x="673.1" y="116.84"/>
 <pinref part="X2" gate="1" pin="2"/>
-<wire x1="718.82" y1="116.84" x2="810.26" y2="116.84" width="0.6096" layer="91"/>
+<wire x1="718.82" y1="116.84" x2="786.13" y2="116.84" width="0.6096" layer="91"/>
+<wire x1="786.13" y1="116.84" x2="810.26" y2="116.84" width="0.6096" layer="91"/>
 <wire x1="811.53" y1="119.38" x2="810.26" y2="119.38" width="0.6096" layer="91"/>
 <wire x1="810.26" y1="119.38" x2="810.26" y2="116.84" width="0.6096" layer="91"/>
@@
 <wire x1="718.82" y1="119.38" x2="718.82" y2="116.84" width="0.1524" layer="91"/>
 <junction x="718.82" y="116.84"/>
+<pinref part="C11" gate="G$1" pin="2"/>
+<wire x1="786.13" y1="167.64" x2="786.13" y2="116.84" width="0.6096" layer="91"/>
+<junction x="786.13" y="116.84"/>
 </segment>
 </net>
@@
 <junction x="673.1" y="224.79"/>
 <pinref part="X3" gate="1" pin="2"/>
-<wire x1="718.82" y1="224.79" x2="810.26" y2="224.79" width="0.6096" layer="91"/>
+<wire x1="718.82" y1="224.79" x2="786.13" y2="224.79" width="0.6096" layer="91"/>
+<wire x1="786.13" y1="224.79" x2="810.26" y2="224.79" width="0.6096" layer="91"/>
 <wire x1="811.53" y1="227.33" x2="810.26" y2="227.33" width="0.6096" layer="91"/>
 <wire x1="810.26" y1="227.33" x2="810.26" y2="224.79" width="0.6096" layer="91"/>
@@
 <wire x1="718.82" y1="222.25" x2="718.82" y2="224.79" width="0.1524" layer="91"/>
 <junction x="718.82" y="224.79"/>
+<pinref part="C11" gate="G$1" pin="1"/>
+<wire x1="786.13" y1="175.26" x2="786.13" y2="224.79" width="0.6096" layer="91"/>
+<junction x="786.13" y="224.79"/>
 </segment>
 </net>

Commit message: Opamp paketleri ve etrafindaki malzemeler kucultuldu.
Parts:
- removed IC9: LM358D, linear:LM358D
- added C12, C13: 150pF, rcl:C-EUC0603
- added C18, C19: (no value), rcl:C-EUC0603
- added IC2: LMV358MMX, linear:LMV358MMX
- added R100, R101, R99: 2k, rcl:R-EU_R0603
- C114, C20, C23, C24: device rcl:C-EUC0805 -> rcl:C-EUC0603
- C14, C15, C21, C22, C38, C39: device rcl:C-EUC1206 -> rcl:C-EUC0603
- IC1: value LM358D -> LMV358MMX; device linear:LM358D -> linear:LMV358MMX
- R10, R16, R17, R9: device rcl:R-EU_R1206 -> rcl:R-EU_R0603
- R18, R4: device rcl:R-EU_R0805 -> rcl:R-EU_R0603
Connections:
- removed net GND_R: R15.1
- removed net V_LEFT: R3.1
- removed net V_RIGHT: R12.1
- new net VA_OUT: C11.1, R12.1, R23.2, U7.IP1-, U7.IP2-, X3.1, X3.2
- new net VB_OUT: C11.2, R15.1, R26.1, U1.IP1-, U1.IP2-, X2.1, X2.2
- new net VIN_SENS_DIFF: C20.1, R4.2
- new net VOUT_DIFF: C23.1, R18.2
- net +3V3: now also IC2P.V+, R100.2; no longer IC9P.V+
- net AGND: now also R7.1
- net DGND: now also C18.2, C19.2, IC2P.V-, R101.1; no longer IC9P.V-
- net GND_L: no longer R7.1
- net N$1: now also C19.1, IC2A.+IN, R100.1, R101.2; no longer C11.2, R26.1, U1.IP1-, U1.IP2-, X2.1, X2.2
- net N$18: now also C13.2
- net N$2: now also IC2A.-IN, IC2A.OUT, R99.1; no longer C11.1, R23.2, U7.IP1-, U7.IP2-, X3.1, X3.2
- net N$20: now also IC1B.+IN; no longer IC9A.+IN
- net N$23: now also C12.1, IC1B.-IN; no longer IC9A.-IN
- net N$25: now also C12.2, IC1B.OUT; no longer IC9A.OUT
- net N$9: now also C13.1
- net VIN: now also R3.1
- net VREF: now also C18.1, R99.2
- net V_LEFT_MESURE: no longer C20.1, R4.2
- net V_RIGHT_MESURE: no longer C23.1, R18.2
Other:
- moved on the sheet: C114

Commit message: Kontrol karti soketleri eklendi.
Giris beslemesini gostermek icin led eklentisi yapildi.
Parts:
- added LED5: (no value), led:LEDCHIPLED_0805
- added R102, R103, R104, R105: (no value), rcl:R-EU_R1206
- added SV1: (no value), con-lsta:FE10-2
- added SV2: (no value), con-lsta:FE08-1
Connections:
- removed net VOUT_DIFF: C23.1, R18.2
- new net FAN: SV1.14
- new net N$54: R102.1, R103.2
- new net N$56: R103.1, R104.2
- new net N$58: R104.1, R105.2
- new net N$68: LED5.A, R105.1
- new net NTC-HS1: SV1.16
- new net NTC-HS2: SV1.18
- new net POWER_IN: SV2.1
- new net VOUT_SENS_DIFF: C23.1, R18.2, SV1.1
- net +3V3: now also SV2.7
- net +5V: now also SV2.5
- net AGND: now also LED5.C, SV2.3
- net DGND: now also SV2.6, SV2.8
- net G11_PWM: now also SV1.2
- net G12_PWM: now also SV1.4
- net G13_PWM: now also SV1.6
- net G14_PWM: now also SV1.8
- net IA_SENS: now also SV1.9
- net IB_SENS: now also SV1.11
- net IIN_SENS: now also SV1.5
- net RELAY1: now also SV1.10
- net RELAY2: now also SV1.12
- net VA_SENS: now also SV1.13
- net VB_SENS: now also SV1.15
- net VDD: now also SV2.4
- net VIN: now also R102.2
- net VIN_SENS: now also SV1.7
- net VIN_SENS_DIFF: now also SV1.3
Other:
- note added: "Kontrol Karti Baglanti Soketleri"
- note removed: "Dijitaller icin Power-Supply modul seklinde yapilacak."

Commit message: Guc hattinda bulunmayan bir cok cap paketi 603 yapildi.
Parts:
- C10, C16, C17, C72, C73, C9: device rcl:C-EUC0805 -> rcl:C-EUC0603
- C139, C140, C144, C145, C25, C26, C75, C76, C87, C88, C89, C90: device rcl:C-USC0805 -> rcl:C-USC0603
- R36, R41: device rcl:R-EU_R0805 -> rcl:R-EU_R0603
Changed lines of the file:
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@@
 <part name="R68" library="rcl" deviceset="R-US_" device="R0603" value="10k"/>
 <part name="R69" library="rcl" deviceset="R-US_" device="R0603" value="10k"/>
-<part name="C25" library="rcl" deviceset="C-US" device="C0805" value="100n"/>
-<part name="C26" library="rcl" deviceset="C-US" device="C0805" value="100n"/>
+<part name="C25" library="rcl" deviceset="C-US" device="C0603" value="100n"/>
+<part name="C26" library="rcl" deviceset="C-US" device="C0603" value="100n"/>
 <part name="D5" library="diode" deviceset="DIODE-" device="DO214AC"/>
 <part name="VCC_1" library="supply2" deviceset="VCC" device=""/>
@@
 <part name="R71" library="rcl" deviceset="R-US_" device="R0603" value="15"/>
 <part name="FB2" library="rcl" deviceset="R-US_" device="R0603" value="180"/>
-<part name="C75" library="rcl" deviceset="C-US" device="C0805" value="100n"/>
-<part name="C76" library="rcl" deviceset="C-US" device="C0805" value="100n"/>
+<part name="C75" library="rcl" deviceset="C-US" device="C0603" value="100n"/>
+<part name="C76" library="rcl" deviceset="C-US" device="C0603" value="100n"/>
 <part name="R73" library="rcl" deviceset="R-US_" device="R0603" value="10k"/>
 <part name="R65" library="rcl" deviceset="R-US_" device="R1206" value="15"/>
@@
 <part name="C85" library="rcl" deviceset="C-US" device="C0603" value="100n"/>
 <part name="C86" library="rcl" deviceset="C-US" device="C0603" value="100n"/>
-<part name="C87" library="rcl" deviceset="C-US" device="C0805" value="100n"/>
-<part name="C88" library="rcl" deviceset="C-US" device="C0805" value="100n"/>
+<part name="C87" library="rcl" deviceset="C-US" device="C0603" value="100n"/>
+<part name="C88" library="rcl" deviceset="C-US" device="C0603" value="100n"/>
 <part name="D6" library="diode" deviceset="DIODE-" device="DO214AC"/>
 <part name="R86" library="rcl" deviceset="R-US_" device="R1206" value="10"/>
@@
 <part name="R88" library="rcl" deviceset="R-US_" device="R0603"/>
 <part name="R67" library="rcl" deviceset="R-US_" device="R0603" value="10k"/>
-<part name="C89" library="rcl" deviceset="C-US" device="C0805" value="100n"/>
-<part name="C90" library="rcl" deviceset="C-US" device="C0805" value="100n"/>
+<part name="C89" library="rcl" deviceset="C-US" device="C0603" value="100n"/>
+<part name="C90" library="rcl" deviceset="C-US" device="C0603" value="100n"/>
 <part name="R89" library="rcl" deviceset="R-US_" device="R1206" value="15"/>
 <part name="C91" library="resistor" deviceset="C-US" device="C1206" value="22p"/>
@@
 <part name="GND12" library="supply1" deviceset="GND" device=""/>
 <part name="C138" library="rcl" deviceset="C-US" device="C0603" value="0.1uF"/>
-<part name="C139" library="rcl" deviceset="C-US" device="C0805" value="0.1uF"/>
-<part name="C140" library="rcl" deviceset="C-US" device="C0805" value="0.1uF"/>
+<part name="C139" library="rcl" deviceset="C-US" device="C0603" value="0.1uF"/>
+<part name="C140" library="rcl" deviceset="C-US" device="C0603" value="0.1uF"/>
 <part name="C141" library="rcl" deviceset="C-US" device="C0805" value="10uF"/>
 <part name="C142" library="rcl" deviceset="C-US" device="C1206" value="22uF"/>
@@
 <part name="P+18" library="supply1" deviceset="VCC" device="" value="+5V"/>
 <part name="C143" library="rcl" deviceset="C-US" device="C0603" value="0.1uF"/>
-<part name="C144" library="rcl" deviceset="C-US" device="C0805" value="0.1uF"/>
-<part name="C145" library="rcl" deviceset="C-US" device="C0805" value="0.1uF"/>
+<part name="C144" library="rcl" deviceset="C-US" device="C0603" value="0.1uF"/>
+<part name="C145" library="rcl" deviceset="C-US" device="C0603" value="0.1uF"/>
 <part name="C146" library="rcl" deviceset="C-US" device="C0805" value="10uF"/>
 <part name="C147" library="rcl" deviceset="C-US" device="C1206" value="22uF"/>
@@
 <part name="C8" library="rcl" library_urn="urn:adsk.eagle:library:334" deviceset="C-EU" device="C1206" package3d_urn="urn:adsk.eagle:package:23618/2" value="https://www.ozdisan.com/passive-components/capacitors/smt-smd-and-mlcc-capacitors/CL31C102JHHNNNE"/>
 <part name="U7" library="enko01" deviceset="ACS712" device=""/>
-<part name="C16" library="rcl" deviceset="C-EU" device="C0805"/>
-<part name="C17" library="rcl" deviceset="C-EU" device="C0805"/>
+<part name="C16" library="rcl" deviceset="C-EU" device="C0603"/>
+<part name="C17" library="rcl" deviceset="C-EU" device="C0603"/>
 <part name="SUPPLY7" library="supply2" deviceset="DGND" device=""/>
 <part name="R19" library="rcl" deviceset="R-EU_" device="R0603"/>
@@
 <part name="Q4" library="transistor-npn" deviceset="BC846*" device="SMD" technology="ALT1" value="1200980569**TRANS SMD NPN MMBTA06 SOT-23 80V 500mA"/>
 <part name="D1" library="diode" deviceset="DIODE-" device="SOD123"/>
-<part name="R36" library="rcl" deviceset="R-EU_" device="R0805"/>
+<part name="R36" library="rcl" deviceset="R-EU_" device="R0603"/>
 <part name="Q6" library="transistor-npn" deviceset="BC846*" device="SMD" technology="ALT1" value="1200980569**TRANS SMD NPN MMBTA06 SOT-23 80V 500mA"/>
 <part name="D2" library="diode" deviceset="DIODE-" device="SOD123"/>
-<part name="R41" library="rcl" deviceset="R-EU_" device="R0805"/>
+<part name="R41" library="rcl" deviceset="R-EU_" device="R0603"/>
 <part name="R32" library="rcl" deviceset="R-EU_" device="0411/12"/>
 <part name="R37" library="rcl" deviceset="R-EU_" device="0411/12"/>
@@
 <part name="+3V22" library="supply1" deviceset="+3V3" device=""/>
 <part name="SUPPLY29" library="supply2" deviceset="+5V" device=""/>
-<part name="C72" library="rcl" deviceset="C-EU" device="C0805"/>
-<part name="C73" library="rcl" deviceset="C-EU" device="C0805"/>
+<part name="C72" library="rcl" deviceset="C-EU" device="C0603"/>
+<part name="C73" library="rcl" deviceset="C-EU" device="C0603"/>
 <part name="SUPPLY61" library="supply2" deviceset="DGND" device=""/>
 <part name="C31" library="rcl" deviceset="CPOL-EU" device="E7.5-18"/>
@@
 <part name="SUPPLY8" library="supply2" deviceset="DGND" device=""/>
 <part name="U1" library="enko01" deviceset="ACS712" device=""/>
-<part name="C9" library="rcl" deviceset="C-EU" device="C0805"/>
-<part name="C10" library="rcl" deviceset="C-EU" device="C0805"/>
+<part name="C9" library="rcl" deviceset="C-EU" device="C0603"/>
+<part name="C10" library="rcl" deviceset="C-EU" device="C0603"/>
 <part name="SUPPLY14" library="supply2" deviceset="DGND" device=""/>
 <part name="R21" library="rcl" deviceset="R-EU_" device="R0603"/>
