File: inverter-1kw.brd (EAGLE design)
At the start: 160 x 100 mm, 257 parts, among them IC1 LMV358MMX, IC2 LMV358MMX, IC5 ISO3082, IC6 25LC080SN, Q2 1200980569**TRANS SMD NPN MMB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, Q3 1200980569**TRANS SMD NPN MMB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, Q4 1200980569**TRANS SMD NPN MMB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, Q6 1200980569**TRANS SMD NPN MMB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, U1 ACS712, U2 STM32F334C6, U3 1039-2088**AM1L-0505SH30-NZ A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, U4 ACS712, U5 SI8230, U6 SI8230, U7 ACS712, X1 MCV3, X2 https://ozdisan.com/connector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, X3 https://ozdisan.com/connector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, X7 https://ozdisan.com/connector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, X8 https://ozdisan.com/connector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

Commit message: ölçüm devresi ve röle kontrol devresi düzenlendi.
Parts:
- removed C43, C44, C47, C53, C54, C74: (no value), rcl:C0805
- removed C45, C52, C55, C56: 100n, rcl:C0805
- removed C46, C57, C69, C70: 4.7u, rcl:C1206
- removed C48: 10n, rcl:C0805
- removed C49: 1u, rcl:C1206
- removed C50, C51: 10p, rcl:C0805
- removed C58, C61: 1200920113**CAP 0805 CER 100NF 50V %20 X7, rcl:C0805
- removed C59: 1019-3202 CAP SMD AL. ELEC 4.7uF 16V %20 85C, rcl:153CLV-0405
- removed C60: 1019-3203 CAP SMD AL. ELEC 10uF 16V %20 85C Dxh(4x5.3mm), rcl:153CLV-0405
- removed D3, D4: https://www.digikey.com/product-detail/en/littelfuse-inc/AQ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, diode:SOD323-W
- removed IC5: ISO3082, enko:ISO3082
- removed IC6: 25LC080SN, microchip:SO-08
- removed JP3: (no value), pinhead:1X06
- removed JP4: (no value), jumper:JP1
- removed JP5, JP6, JP7, JP8: (no value), pinhead:1X02
- removed L4: ACM2012-900--2P-T002, enko:ACM2012-900--2P-T002
- removed LED1, LED2, LED3, LED4: (no value), led:1206
- removed Q1: (no value), crystal:SM49
- removed Q2, Q3: 1200980569**TRANS SMD NPN MMBTA06 SOT-23 80V 500mA, transistor-npn:SOT23
- removed R28, R33, R34, R35, R38, R55, R64: (no value), rcl:R0805
- removed R29: 4k7, rcl:R0805
- removed R30: 10k, rcl:R0805
- removed R31, R39, R40: 470R, rcl:R0805
- removed R44, R45, R46, R47, R48, R49, R52, R53, R54, R61: (no value), rcl:R0603
- removed R50: 1200970601 RES 1206 10R %5 1/4W, rcl:R1206
- removed R51, R58: NC, rcl:R0805
- removed R56: 1029-3164**RES 1206 120R %1, rcl:R1206
- removed R62, R63: 1200970601**RES 1206 10R %5 1/4W, rcl:R1206
- removed U2: STM32F334C6, enko01:LQFP48
- removed U3: 1039-2088**AM1L-0505SH30-NZ AIMTEC 85C SMD DC-DC Converter, enkohasip:LF101ESI
- removed X1: MCV3, con-phoenix-381_l:MCV3
- moved LED5 294.3 mm to (6.53, 61.8), turned to 90 degrees
- moved R105 293.4 mm to (8.97, 63.5)
- moved R104 292.1 mm to (8.98, 65.6), turned to 180 degrees
- moved R103 290.9 mm to (8.98, 67.6)
- moved R102 289.7 mm to (8.98, 69.7), turned to 180 degrees
- moved R96 227.4 mm to (3.94, 63.5), turned to 180 degrees
- moved R95 222.3 mm to (3.94, 65.6)
- moved R94 217.2 mm to (3.93, 67.6), turned to 180 degrees
- moved SV1 217.0 mm to (-50.8, 54.9), turned to 270 degrees
- moved R93 212.1 mm to (3.93, 69.7)
- moved RL2 202.0 mm to (14.4, 81.4)
- moved RL1 201.9 mm to (14.5, 91.9)
- moved C138 180.3 mm to (30.4, 40.9), flipped to the bottom, turned to 270 degrees
- moved C139 147.7 mm to (30.4, 46.8), flipped to the bottom, turned to 270 degrees
- moved DC1 133.9 mm to (28.8, 44.1), turned to 90 degrees
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Connections:
- removed net +15V: JP7.2, JP8.2
- removed net +5V/1: C60.+, C61.2, IC5.16, R51.1, U3.8
- removed net 485A: D3.C, L4.3, X1.1
- removed net 485B: L4.1, R62.2
- removed net FAN1_CONT: R39.1, U2.21
- removed net FAN2_CONT: R40.1, U2.22
- removed net FRAM_CS: R64.2, U2.42
- removed net FRAM_HOLD: IC6.7, R55.1, U2.33
- removed net FRAM_WP: IC6.3, U2.38
- removed net G21_PWM: U2.25
- removed net G22_PWM: U2.26
- removed net G23_PWM: U2.27
- removed net G24_PWM: U2.28
- removed net I_LEFT_DC: R61.1
- removed net I_RIGHT_AC: R48.1
- removed net I_RIGHT_DC: R46.1
- removed net LED1: LED1.C, U2.4
- removed net LED2: LED2.C, U2.3
- removed net LED3: LED3.C, U2.2
- removed net LED4: LED4.C, U2.46
- removed net MISO: IC6.2, U2.40
- removed net MOSI: IC6.5, U2.41
- removed net N$14: L4.2, R63.1
- removed net N$22: R28.2, U2.6
- removed net N$33: C51.2, Q1.1, R28.1
- removed net N$34: C50.2, Q1.2, U2.5
- removed net N$35: IC5.13, R56.1, R58.2, R62.1
- removed net N$36: IC5.12, R51.2, R56.2, R63.2
- removed net N$37: JP3.6, R29.1
- removed net N$38: JP4.1, R30.2, U2.44
- removed net N$39: JP4.2, R31.1
- removed net N$40: LED2.A, R35.2
- removed net N$41: C53.1, R47.2, U2.18
- removed net N$42: LED1.A, R34.2
- removed net N$43: LED4.A, R33.2
- removed net N$46: C55.1, JP6.2, R49.2, R53.1
- removed net N$47: C54.1, R48.2, U2.19
- removed net N$48: LED3.A, R38.2
- removed net N$49: C43.1, R44.2, U2.14
- removed net N$50: C44.1, R45.2, U2.15
- removed net N$53: C47.1, R46.2, U2.16
- removed net N$59: JP8.1, Q3.3
- removed net N$60: JP7.1, Q2.3
- removed net N$61: C56.1, JP5.2, R52.2, R54.1
- removed net N$62: Q2.1, R39.2
- removed net N$63: C69.1, IC6.1, R64.1
- removed net N$64: Q3.1, R40.2
- removed net N$65: D4.C, L4.4, X1.3
- removed net N$66: C74.1, R61.2, U2.10
- removed net N$67: D3.A, D4.A, R50.2, X1.2
- removed net NRST: C52.1, JP3.2, U2.7
- removed net NTC1: R53.2, U2.17
- removed net NTC2: R54.2, U2.20
- removed net SGND: C60.-, C61.1, IC5.10, IC5.15, IC5.9, R50.1, R58.1, U3.5
- removed net SWCLK: JP3.5, U2.37
- removed net SWDIO: JP3.3, U2.34
- removed net SWO: IC6.6, JP3.1, U2.39
- removed net USART2_DE: IC5.4, IC5.5, U2.11
- removed net USART2_RX: IC5.3, U2.13
- removed net USART2_TX: IC5.6, U2.12
- removed net VBAT: U2.1
- removed net V_LEFT_MESURE: R44.1
- removed net V_RIGHT_MESURE: R45.1
- net +3V3: no longer C45.1, C46.1, C48.1, C49.1, C57.1, C58.2, C70.1, IC5.1, IC6.8, JP5.1, JP6.1, R29.2, R31.2, R33.1, R34.1, R35.1, R38.1, R55.2, U2.24, U2.36, U2.48, U2.9
- net +5V: no longer C59.+, U3.2
- net DGND: no longer C43.2, C44.2, C45.2, C46.2, C47.2, C48.2, C49.2, C50.1, C51.1, C52.2, C53.2, C54.2, C55.2, C56.2, C57.2, C58.1, C59.-, C69.2, C70.2, C74.2, IC5.2, IC5.7, IC5.8, IC6.4, JP3.4, Q2.2, Q3.2, R30.1, R49.1, R52.1, U2.23, U2.35, U2.47, U2.8, U3.1
- net G11_PWM: no longer U2.29
- net G12_PWM: no longer U2.30
- net G13_PWM: no longer U2.31
- net G14_PWM: no longer U2.32
- net IB_SENS: no longer R47.1
- net RELAY1: no longer U2.45
- net RELAY2: no longer U2.43
Routing:
- net V_IN: track 16.6 -> 59.9 mm
- net VSUPPLY+: track 0.00 -> 35.4 mm
- net N$51: track 20.4 -> 4.45 mm
- net DGND: track 5.58 -> 12.8 mm
- net N$44: track 7.83 -> 14.3 mm
- net N$70: track 5.84 -> 0.01 mm
- net VIN: track 0.00 -> 5.10 mm
- net N$45: track 0.00 -> 2.50 mm
- net N$56: track 0.00 -> 2.07 mm
- net N$31: track 0.00 -> 2.05 mm
- net N$58: track 0.00 -> 2.05 mm
- net VIN_SENS: track 0.00 -> 2.05 mm
- net N$54: track 0.00 -> 2.05 mm
- net N$4: track 0.00 -> 2.05 mm
- net N$52: track 0.00 -> 1.93 mm
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